Commit message: fix pandar urdf

File: urdf/hesai.urdf.xacro (robot description, xacro)
@@ -1,4 +1,4 @@
 <?xml version="1.0"?>
-<!-- Copyright 2020 University of Oxford
+<!-- Copyright 2022 University of Oxford
    Licensed under the Apache License, Version 2.0 (the "License");
    you may not use this file except in compliance with the License.
@@ -46,10 +46,11 @@
     </collision>
   </link>
-  <link name="hesai_origin"/>
-  <joint name="hesai_base_to_origin" type="fixed">
+  <link name="pandar"/>
+  <joint name="hesai_base_to_pandar" type="fixed">
     <!-- See page 12 of User Manual -->
-    <origin xyz="0.0 0.0 46.4e-3" rpy="0.0 0.0 0.0"/>
+    <!-- note that the X axis points left. See manual page 11 -->
+    <origin xyz="0.0 0.0 46.4e-3" rpy="0.0 0.0 ${pi/2}"/>
     <parent link="hesai_base"/>
-    <child link="hesai_origin" />
+    <child link="pandar" />
   </joint>
   <!-- TODO implement gazebo plugin loading if simulation is true -->

File: urdf/hesai_standalone.urdf.xacro (robot description, xacro)
@@ -1,4 +1,4 @@
 <?xml version="1.0"?>
-<!-- Copyright 2020 University of Oxford
+<!-- Copyright 2022 University of Oxford
    Licensed under the Apache License, Version 2.0 (the "License");
    you may not use this file except in compliance with the License.

Commit message: make the lidar frame name parametric

File: urdf/hesai.urdf.xacro (robot description, xacro)
@@ -14,5 +14,5 @@
 <robot name="hesai" xmlns:xacro="http://www.ros.org/wiki/xacro">
 <xacro:arg name="simulation" default="false" />
-<xacro:macro name="hesai_device" params="parent *origin name:=pandar_xt32_lidar simulation:=false">
+<xacro:macro name="hesai_device" params="parent *origin name:=pandar_xt32_lidar simulation:=false lidar_frame:=pandar">
   <joint name="${parent}_to_hesai" type="fixed">
     <xacro:insert_block name="origin"/>
@@ -46,5 +46,5 @@
     </collision>
   </link>
-  <link name="pandar"/>
+  <link name="${lidar_frame}"/>
   <joint name="hesai_base_to_pandar" type="fixed">
     <!-- See page 12 of User Manual -->
@@ -52,5 +52,5 @@
     <origin xyz="0.0 0.0 46.4e-3" rpy="0.0 0.0 ${pi/2}"/>
     <parent link="hesai_base"/>
-    <child link="pandar" />
+    <child link="${lidar_frame}" />
   </joint>
   <!-- TODO implement gazebo plugin loading if simulation is true -->

Commit message: fix: Adapt Hesai QT64 default orientation

File: urdf/hesai.urdf.xacro (robot description, xacro)
@@ -50,5 +50,5 @@
     <!-- See page 12 of User Manual -->
     <!-- note that the X axis points left. See manual page 11 -->
-    <origin xyz="0.0 0.0 50.4e-3" rpy="0.0 0.0 0.0"/>
+    <origin xyz="0.0 0.0 50.4e-3" rpy="0.0 0.0 ${pi}"/>
     <parent link="hesai_base"/>
     <child link="${lidar_frame}" />
