Commit message: fix: Add consistent frames according to manufacturer manual for QT64 and XT32 lidars

File: urdf/hesai_qt64_standalone.urdf.xacro (robot description, xacro)
@@ -11,10 +11,11 @@
    limitations under the License. -->
 <robot name="hesai" xmlns:xacro="http://www.ros.org/wiki/xacro">
-  <xacro:include filename="$(find hesai_description)/urdf/hesai.urdf.xacro" />
+  <xacro:include filename="$(find hesai_description)/urdf/hesai_qt64.urdf.xacro" />
   <xacro:arg name="simulation" default="false" />
+  <xacro:arg name="use_gpu" default="true" />
   <!-- Dummy link  -->
   <link name="base"/>
-  <xacro:hesai_device parent="base" simulation="$(arg simulation)">
+  <xacro:hesai_qt64_device parent="base" simulation="$(arg simulation)" use_gpu="$(arg use_gpu)" >
     <origin xyz="0 0 0" rpy="0 0 0" />
-  </xacro:hesai_device>
+  </xacro:hesai_qt64_device>
 </robot>

File: urdf/hesai_xt32.urdf.xacro (robot description, xacro)
@@ -12,7 +12,8 @@
 -->
 <!-- Hesai PandarXT-32 Lidar Sensor -->
-<robot name="hesai" xmlns:xacro="http://www.ros.org/wiki/xacro">
+<robot name="hesai_xt32" xmlns:xacro="http://www.ros.org/wiki/xacro">
 <xacro:arg name="simulation" default="false" />
-<xacro:macro name="hesai_device" params="parent *origin name:=pandar_xt32_lidar simulation:=false lidar_frame:=pandar">
+<xacro:arg name="use_gpu" default="true"/>
+<xacro:macro name="hesai_xt32_device" params="parent *origin name:=pandar_xt32_lidar simulation:=false lidar_frame:=pandar use_gpu:=true">
   <joint name="${parent}_to_hesai" type="fixed">
     <xacro:insert_block name="origin"/>
@@ -48,11 +49,17 @@
   <link name="${lidar_frame}"/>
   <joint name="hesai_base_to_pandar" type="fixed">
-    <!-- See page 12 of User Manual -->
+    <!-- See page 12 of XT64 User Manual -->
     <!-- note that the X axis points left. See manual page 11 -->
-    <origin xyz="0.0 0.0 50.4e-3" rpy="0.0 0.0 0.0"/>
+    <origin xyz="0.0 0.0 46.4e-3" rpy="0.0 0.0 ${pi/2}"/>
     <parent link="hesai_base"/>
     <child link="${lidar_frame}" />
   </joint>
-  <!-- TODO implement gazebo plugin loading if simulation is true -->
+  <xacro:if value="${simulation}">
+    <xacro:include filename="$(find hesai_description)/urdf/gazebo.urdf.xacro"/>
+    <xacro:hesai_gazebo lidar_frame="${lidar_frame}" topic_name="/hesai/pandar" min_range="0.4" max_range="80.0"
+      min_horizontal_angle="-180.0" max_horizontal_angle="180.0" min_vertical_angle="-16.0" max_vertical_angle="15.0"
+      hz="10" samples="2000" lasers="32" collision_range="0.3" noise="0.008" use_gpu="${use_gpu}"
+    />
+  </xacro:if>
 </xacro:macro>
 </robot>
