Commit message: fix: Add tf prefix for including multiple Hesai models into the same URDF

File: urdf/gazebo.urdf.xacro (robot description, xacro)
@@ -12,5 +12,5 @@
    limitations under the License.
 -->
-  <xacro:macro name="hesai_gazebo" params="lidar_frame:=pandar topic_name=/hesai/pandar
+  <xacro:macro name="hesai_gazebo" params="prefix lidar_frame:=pandar topic_name=/hesai/pandar
                min_range:=0.4 max_range:=80.0 min_horizontal_angle:=-180.0 max_horizontal_angle:=180.0
                min_vertical_angle:=-16.0 max_vertical_angle:=15.0 hz:=10 samples:=2000 lasers:=32
@@ -25,5 +25,5 @@
         <xacro:property name="laser_plugin" value="libgazebo_ros_velodyne_laser.so" />
       </xacro:unless>
-      <sensor type="${ray_type}" name="hesai_sensor">
+      <sensor type="${ray_type}" name="${prefix}hesai_sensor">
         <pose>0 0 0 0 0 0</pose>
         <visualize>${visualize}</visualize>
@@ -55,5 +55,5 @@
           </noise>
         </ray>
-        <plugin name="gazebo_ros_laser_controller" filename="${laser_plugin}">
+        <plugin name="${prefix}gazebo_ros_laser_controller" filename="${laser_plugin}">
           <topicName>${topic_name}</topicName>
           <frameName>${lidar_frame}</frameName>

File: urdf/hesai_qt64.urdf.xacro (robot description, xacro)
@@ -15,11 +15,13 @@
 <xacro:arg name="simulation" default="false"/>
 <xacro:arg name="use_gpu" default="true"/>
-<xacro:macro name="hesai_qt64_device" params="parent *origin name:=pandar_xt32_lidar simulation:=false lidar_frame:=pandar use_gpu:=true">
-  <joint name="${parent}_to_hesai" type="fixed">
+<xacro:macro name="hesai_qt64_device" params="parent *origin prefix:='' name:=pandar_qt64_lidar
+                                              topic_name:=/hesai/pandar
+                                              simulation:=false lidar_frame:=pandar use_gpu:=true">
+  <joint name="${parent}_to_${prefix}hesai" type="fixed">
     <xacro:insert_block name="origin"/>
     <parent link="${parent}" />
-    <child link="hesai_base" />
+    <child link="${prefix}hesai_base" />
   </joint>
-  <link name="hesai_base">
+  <link name="${prefix}hesai_base">
     <visual>
       <origin xyz="0 0 0" rpy="0 0 0" />
@@ -48,14 +50,14 @@
   </link>
   <link name="${lidar_frame}"/>
-  <joint name="hesai_base_to_pandar" type="fixed">
+  <joint name="${prefix}hesai_base_to_pandar" type="fixed">
     <!-- See page 12 of QT64 User Manual -->
     <!-- note that the X axis points left. See manual page 11 -->
     <origin xyz="0.0 0.0 50.4e-3" rpy="0.0 0.0 ${pi/2}"/>
-    <parent link="hesai_base"/>
+    <parent link="${prefix}hesai_base"/>
     <child link="${lidar_frame}" />
   </joint>
   <xacro:if value="${simulation}">
     <xacro:include filename="$(find hesai_description)/urdf/gazebo.urdf.xacro"/>
-    <xacro:hesai_gazebo lidar_frame="${lidar_frame}" topic_name="/hesai/pandar" min_range="0.1" max_range="20.0"
+    <xacro:hesai_gazebo prefix="${prefix}" lidar_frame="${lidar_frame}" topic_name="${topic_name}" min_range="0.1" max_range="20.0"
       min_horizontal_angle="-180.0" max_horizontal_angle="180.0" min_vertical_angle="-52.1" max_vertical_angle="52.1"
       hz="10" samples="600" lasers="64" collision_range="0.3" noise="0.008" use_gpu="${use_gpu}"

File: urdf/hesai_qt64_standalone.urdf.xacro (robot description, xacro)
@@ -12,9 +12,12 @@
 <robot name="hesai" xmlns:xacro="http://www.ros.org/wiki/xacro">
   <xacro:include filename="$(find hesai_description)/urdf/hesai_qt64.urdf.xacro" />
+  <xacro:arg name="prefix" default="" />
   <xacro:arg name="simulation" default="false" />
   <xacro:arg name="use_gpu" default="true" />
   <!-- Dummy link  -->
   <link name="base"/>
-  <xacro:hesai_qt64_device parent="base" simulation="$(arg simulation)" use_gpu="$(arg use_gpu)" >
+  <xacro:hesai_qt64_device parent="base" prefix="$(arg prefix)"
+    lidar_frame="$(arg prefix)pandar"
+    simulation="$(arg simulation)" use_gpu="$(arg use_gpu)" >
     <origin xyz="0 0 0" rpy="0 0 0" />
   </xacro:hesai_qt64_device>

File: urdf/hesai_xt32.urdf.xacro (robot description, xacro)
@@ -15,11 +15,13 @@
 <xacro:arg name="simulation" default="false" />
 <xacro:arg name="use_gpu" default="true"/>
-<xacro:macro name="hesai_xt32_device" params="parent *origin name:=pandar_xt32_lidar simulation:=false lidar_frame:=pandar use_gpu:=true">
-  <joint name="${parent}_to_hesai" type="fixed">
+<xacro:macro name="hesai_xt32_device" params="parent *origin prefix:='' name:=pandar_xt32_lidar
+                                              topic_name:=/hesai/pandar
+                                              simulation:=false lidar_frame:=pandar use_gpu:=true">
+  <joint name="${parent}_to_${prefix}hesai" type="fixed">
     <xacro:insert_block name="origin"/>
     <parent link="${parent}" />
-    <child link="hesai_base" />
+    <child link="${prefix}hesai_base" />
   </joint>
-  <link name="hesai_base">
+  <link name="${prefix}hesai_base">
     <visual>
       <origin xyz="0 0 0" rpy="0 0 0" />
@@ -48,14 +50,14 @@
   </link>
   <link name="${lidar_frame}"/>
-  <joint name="hesai_base_to_pandar" type="fixed">
+  <joint name="${prefix}hesai_base_to_pandar" type="fixed">
     <!-- See page 12 of XT64 User Manual -->
     <!-- note that the X axis points left. See manual page 11 -->
     <origin xyz="0.0 0.0 46.4e-3" rpy="0.0 0.0 ${pi/2}"/>
-    <parent link="hesai_base"/>
+    <parent link="${prefix}hesai_base"/>
     <child link="${lidar_frame}" />
   </joint>
   <xacro:if value="${simulation}">
     <xacro:include filename="$(find hesai_description)/urdf/gazebo.urdf.xacro"/>
-    <xacro:hesai_gazebo lidar_frame="${lidar_frame}" topic_name="/hesai/pandar" min_range="0.4" max_range="80.0"
+    <xacro:hesai_gazebo prefix="${prefix}" lidar_frame="${lidar_frame}" topic_name="${topic_name}" min_range="0.4" max_range="80.0"
       min_horizontal_angle="-180.0" max_horizontal_angle="180.0" min_vertical_angle="-16.0" max_vertical_angle="15.0"
       hz="10" samples="2000" lasers="32" collision_range="0.3" noise="0.008" use_gpu="${use_gpu}"

File: urdf/hesai_xt32_standalone.urdf.xacro (robot description, xacro)
@@ -12,9 +12,12 @@
 <robot name="hesai" xmlns:xacro="http://www.ros.org/wiki/xacro">
   <xacro:include filename="$(find hesai_description)/urdf/hesai_xt32.urdf.xacro" />
+  <xacro:arg name="prefix" default="" />
   <xacro:arg name="simulation" default="false" />
   <xacro:arg name="use_gpu" default="true" />
   <!-- Dummy link  -->
   <link name="base"/>
-  <xacro:hesai_xt32_device parent="base" simulation="$(arg simulation)" use_gpu="$(arg use_gpu)" >
+  <xacro:hesai_xt32_device parent="base" prefix="$(arg prefix)"
+    lidar_frame="$(arg prefix)pandar"
+    simulation="$(arg simulation)" use_gpu="$(arg use_gpu)" >
     <origin xyz="0 0 0" rpy="0 0 0" />
   </xacro:hesai_xt32_device>

Commit message: refactor: Port Hesai description to ROS 2

File: urdf/gazebo.urdf.xacro (robot description, xacro)
@@ -1,15 +1,4 @@
 <?xml version="1.0"?>
 <robot xmlns:xacro="http://www.ros.org/wiki/xacro">
-<!-- Copyright 2024 University of Oxford
-   Licensed under the Apache License, Version 2.0 (the "License");
-   you may not use this file except in compliance with the License.
-   You may obtain a copy of the License at
-       http://www.apache.org/licenses/LICENSE-2.0
-   Unless required by applicable law or agreed to in writing, software
-   distributed under the License is distributed on an "AS IS" BASIS,
-   WITHOUT WARRANTIES OR CONDITIONS OF ANY KIND, either express or implied.
-   See the License for the specific language governing permissions and
-   limitations under the License.
--->
   <xacro:macro name="hesai_gazebo" params="prefix lidar_frame:=pandar topic_name=/hesai/pandar
                min_range:=0.4 max_range:=80.0 min_horizontal_angle:=-180.0 max_horizontal_angle:=180.0

File: urdf/hesai_qt64.urdf.xacro (robot description, xacro)
@@ -1,67 +1,49 @@
 <?xml version="1.0"?>
-<!-- Copyright 2022 University of Oxford
-   Licensed under the Apache License, Version 2.0 (the "License");
-   you may not use this file except in compliance with the License.
-   You may obtain a copy of the License at
-       http://www.apache.org/licenses/LICENSE-2.0
-   Unless required by applicable law or agreed to in writing, software
-   distributed under the License is distributed on an "AS IS" BASIS,
-   WITHOUT WARRANTIES OR CONDITIONS OF ANY KIND, either express or implied.
-   See the License for the specific language governing permissions and
-   limitations under the License.
--->
-<!-- Hesai PandarQT-64 Lidar Sensor -->
 <robot name="hesai_qt64" xmlns:xacro="http://www.ros.org/wiki/xacro">
-<xacro:arg name="simulation" default="false"/>
-<xacro:arg name="use_gpu" default="true"/>
-<xacro:macro name="hesai_qt64_device" params="parent *origin prefix:='' name:=pandar_qt64_lidar
-                                              topic_name:=/hesai/pandar
-                                              simulation:=false lidar_frame:=pandar use_gpu:=true">
-  <joint name="${parent}_to_${prefix}hesai" type="fixed">
-    <xacro:insert_block name="origin"/>
-    <parent link="${parent}" />
-    <child link="${prefix}hesai_base" />
-  </joint>
-  <link name="${prefix}hesai_base">
-    <visual>
-      <origin xyz="0 0 0" rpy="0 0 0" />
-      <!-- If mesh is not available: -->
-      <!--origin xyz="0 0 38.0e-3" rpy="0 0 0" /-->
-      <geometry>
-        <!-- If mesh is not available: -->
-        <!--cylinder radius="51.500e-3" length="76.0e-3" /-->
-        <mesh filename="package://hesai_description/urdf/meshes/PandarQT64_model.dae" />
-      </geometry>
-    </visual>
-    <inertial>
-      <!-- CoM taken from CAD assuming constant density and mass 0.807 (best approximation available to real mass) -->
-      <origin xyz="-0.015e-3 0.0 37.494e-3" rpy="0 0 0" />
-      <!-- mass taken from Hesai datasheet -->
-      <mass value="0.807" />
-      <!-- Inertia tensor from CAD assuming constant density and mass 0.807 (best approximation vailable to real mass) -->
-      <inertia ixx="886.81e-6" ixy="5.802e-11" ixz="-0.34e-6" iyy="898.12e-6" iyz="-0.014e-6" izz="1004.287e-6" />
-    </inertial>
-    <collision>
-      <origin xyz="0 0 38.0e-3"/>
-      <geometry>
-        <cylinder radius="51.500e-3" length="76.0e-3" />
-      </geometry>
-    </collision>
-  </link>
-  <link name="${lidar_frame}"/>
-  <joint name="${prefix}hesai_base_to_pandar" type="fixed">
-    <!-- See page 12 of QT64 User Manual -->
-    <!-- note that the X axis points left. See manual page 11 -->
-    <origin xyz="0.0 0.0 50.4e-3" rpy="0.0 0.0 ${pi/2}"/>
-    <parent link="${prefix}hesai_base"/>
-    <child link="${lidar_frame}" />
-  </joint>
-  <xacro:if value="${simulation}">
-    <xacro:include filename="$(find hesai_description)/urdf/gazebo.urdf.xacro"/>
-    <xacro:hesai_gazebo prefix="${prefix}" lidar_frame="${lidar_frame}" topic_name="${topic_name}" min_range="0.1" max_range="20.0"
-      min_horizontal_angle="-180.0" max_horizontal_angle="180.0" min_vertical_angle="-52.1" max_vertical_angle="52.1"
-      hz="10" samples="600" lasers="64" collision_range="0.3" noise="0.008" use_gpu="${use_gpu}"
-    />
-  </xacro:if>
-</xacro:macro>
+  <xacro:arg name="simulation" default="false"/>
+  <xacro:arg name="use_gpu" default="true"/>
+  <xacro:macro name="hesai_qt64" params="parent *origin prefix:='' name:=pandar_qt64
+                                         topic_name:=/hesai/pandar
+                                         simulation:=false lidar_frame:=pandar use_gpu:=true">
+    <joint name="${parent}_to_${prefix}hesai" type="fixed">
+      <xacro:insert_block name="origin"/>
+      <parent link="${parent}" />
+      <child link="${prefix}hesai_base" />
+    </joint>
+    <link name="${prefix}hesai_base">
+      <visual>
+        <origin xyz="0 0 0" rpy="0 0 0" />
+        <geometry>
+          <mesh filename="file://$(find hesai_description)/meshes/visual/qt64.dae" />
+        </geometry>
+      </visual>
+      <inertial>
+        <!-- TODO Still correspond to values of XT32 -->
+        <origin xyz="-0.015e-3 0.0 37.494e-3" rpy="0 0 0" />
+        <mass value="0.807" />
+        <inertia ixx="886.81e-6" ixy="5.802e-11" ixz="-0.34e-6" iyy="898.12e-6" iyz="-0.014e-6" izz="1004.287e-6" />
+      </inertial>
+      <collision>
+        <origin xyz="0 0 38.0e-3"/>
+        <geometry>
+          <cylinder radius="51.500e-3" length="76.0e-3" />
+        </geometry>
+      </collision>
+    </link>
+    <link name="${lidar_frame}"/>
+    <joint name="${prefix}hesai_base_to_${lidar_frame}" type="fixed">
+      <!-- See page 12 of QT64 user manual -->
+      <!-- Note that the X axis points left See manual page 11 -->
+      <origin xyz="0.0 0.0 50.4e-3" rpy="0.0 0.0 ${pi/2}"/>
+      <parent link="${prefix}hesai_base"/>
+      <child link="${lidar_frame}" />
+    </joint>
+    <xacro:if value="${simulation}">
+      <xacro:include filename="$(find hesai_description)/urdf/gazebo.urdf.xacro"/>
+      <xacro:hesai_gazebo prefix="${prefix}" lidar_frame="${lidar_frame}" topic_name="${topic_name}" min_range="0.1" max_range="20.0"
+        min_horizontal_angle="-180.0" max_horizontal_angle="180.0" min_vertical_angle="-52.1" max_vertical_angle="52.1"
+        hz="10" samples="600" lasers="64" collision_range="0.3" noise="0.008" use_gpu="${use_gpu}"
+      />
+    </xacro:if>
+  </xacro:macro>
 </robot>

File: urdf/hesai_qt64_standalone.urdf.xacro (robot description, xacro)
@@ -1,24 +1,12 @@
 <?xml version="1.0"?>
-<!-- Copyright 2022 University of Oxford
-   Licensed under the Apache License, Version 2.0 (the "License");
-   you may not use this file except in compliance with the License.
-   You may obtain a copy of the License at
-       http://www.apache.org/licenses/LICENSE-2.0
-   Unless required by applicable law or agreed to in writing, software
-   distributed under the License is distributed on an "AS IS" BASIS,
-   WITHOUT WARRANTIES OR CONDITIONS OF ANY KIND, either express or implied.
-   See the License for the specific language governing permissions and
-   limitations under the License. -->
 <robot name="hesai" xmlns:xacro="http://www.ros.org/wiki/xacro">
-  <xacro:include filename="$(find hesai_description)/urdf/hesai_qt64.urdf.xacro" />
   <xacro:arg name="prefix" default="" />
   <xacro:arg name="simulation" default="false" />
   <xacro:arg name="use_gpu" default="true" />
-  <!-- Dummy link  -->
+  <xacro:include filename="$(find hesai_description)/urdf/hesai_qt64.urdf.xacro" />
   <link name="base"/>
-  <xacro:hesai_qt64_device parent="base" prefix="$(arg prefix)"
-    lidar_frame="$(arg prefix)pandar"
-    simulation="$(arg simulation)" use_gpu="$(arg use_gpu)" >
+  <xacro:hesai_qt64 parent="base" prefix="$(arg prefix)" lidar_frame="$(arg prefix)pandar"
+                    simulation="$(arg simulation)" use_gpu="$(arg use_gpu)" >
     <origin xyz="0 0 0" rpy="0 0 0" />
-  </xacro:hesai_qt64_device>
+  </xacro:hesai_qt64>
 </robot>

File: urdf/hesai_xt32.urdf.xacro (robot description, xacro)
@@ -1,67 +1,50 @@
 <?xml version="1.0"?>
-<!-- Copyright 2022 University of Oxford
-   Licensed under the Apache License, Version 2.0 (the "License");
-   you may not use this file except in compliance with the License.
-   You may obtain a copy of the License at
-       http://www.apache.org/licenses/LICENSE-2.0
-   Unless required by applicable law or agreed to in writing, software
-   distributed under the License is distributed on an "AS IS" BASIS,
-   WITHOUT WARRANTIES OR CONDITIONS OF ANY KIND, either express or implied.
-   See the License for the specific language governing permissions and
-   limitations under the License.
--->
-<!-- Hesai PandarXT-32 Lidar Sensor -->
 <robot name="hesai_xt32" xmlns:xacro="http://www.ros.org/wiki/xacro">
-<xacro:arg name="simulation" default="false" />
-<xacro:arg name="use_gpu" default="true"/>
-<xacro:macro name="hesai_xt32_device" params="parent *origin prefix:='' name:=pandar_xt32_lidar
-                                              topic_name:=/hesai/pandar
-                                              simulation:=false lidar_frame:=pandar use_gpu:=true">
-  <joint name="${parent}_to_${prefix}hesai" type="fixed">
-    <xacro:insert_block name="origin"/>
-    <parent link="${parent}" />
-    <child link="${prefix}hesai_base" />
-  </joint>
-  <link name="${prefix}hesai_base">
-    <visual>
-      <origin xyz="0 0 0" rpy="0 0 0" />
-      <!-- If mesh is not available: -->
-      <!--origin xyz="0 0 38.0e-3" rpy="0 0 0" /-->
-      <geometry>
-        <!-- If mesh is not available: -->
-        <!--cylinder radius="51.500e-3" length="76.0e-3" /-->
-        <mesh filename="package://hesai_description/urdf/meshes/PandarXT_Model.dae" />
-      </geometry>
-    </visual>
-    <inertial>
-      <!-- CoM taken from CAD assuming constant density and mass 0.807 (best approximation available to real mass) -->
-      <origin xyz="-0.015e-3 0.0 37.494e-3" rpy="0 0 0" />
-      <!-- mass taken from Hesai datasheet -->
-      <mass value="0.807" />
-      <!-- Inertia tensor from CAD assuming constant density and mass 0.807 (best approximation vailable to real mass) -->
-      <inertia ixx="886.81e-6" ixy="5.802e-11" ixz="-0.34e-6" iyy="898.12e-6" iyz="-0.014e-6" izz="1004.287e-6" />
-    </inertial>
-    <collision>
-      <origin xyz="0 0 38.0e-3"/>
-      <geometry>
-        <cylinder radius="51.500e-3" length="76.0e-3" />
-      </geometry>
-    </collision>
-  </link>
-  <link name="${lidar_frame}"/>
-  <joint name="${prefix}hesai_base_to_pandar" type="fixed">
-    <!-- See page 12 of XT64 User Manual -->
-    <!-- note that the X axis points left. See manual page 11 -->
-    <origin xyz="0.0 0.0 46.4e-3" rpy="0.0 0.0 ${pi/2}"/>
-    <parent link="${prefix}hesai_base"/>
-    <child link="${lidar_frame}" />
-  </joint>
-  <xacro:if value="${simulation}">
-    <xacro:include filename="$(find hesai_description)/urdf/gazebo.urdf.xacro"/>
-    <xacro:hesai_gazebo prefix="${prefix}" lidar_frame="${lidar_frame}" topic_name="${topic_name}" min_range="0.4" max_range="80.0"
-      min_horizontal_angle="-180.0" max_horizontal_angle="180.0" min_vertical_angle="-16.0" max_vertical_angle="15.0"
-      hz="10" samples="2000" lasers="32" collision_range="0.3" noise="0.008" use_gpu="${use_gpu}"
-    />
-  </xacro:if>
-</xacro:macro>
+  <xacro:arg name="simulation" default="false" />
+  <xacro:arg name="use_gpu" default="true"/>
+  <xacro:macro name="hesai_xt32" params="parent *origin prefix:='' name:=hesai_xt32
+                                        topic_name:=/hesai/pandar
+                                        simulation:=false lidar_frame:=pandar use_gpu:=true">
+    <joint name="${parent}_to_${prefix}hesai" type="fixed">
+      <xacro:insert_block name="origin"/>
+      <parent link="${parent}" />
+      <child link="${prefix}hesai_base" />
+    </joint>
+    <link name="${prefix}hesai_base">
+      <visual>
+        <origin xyz="0 0 0" rpy="0 0 0" />
+        <geometry>
+          <mesh filename="file://$(find hesai_description)/meshes/visual/xt32.dae" />
+        </geometry>
+      </visual>
+      <inertial>
+        <!-- Taken from CAD assuming constant density and mass 0.807 -->
+        <origin xyz="-0.015e-3 0.0 37.494e-3" rpy="0 0 0" />
+        <!-- Taken from datasheet -->
+        <mass value="0.807" />
+        <!-- Taken from CAD assuming constant density and mass 0.807 -->
+        <inertia ixx="886.81e-6" ixy="5.802e-11" ixz="-0.34e-6" iyy="898.12e-6" iyz="-0.014e-6" izz="1004.287e-6" />
+      </inertial>
+      <collision>
+        <origin xyz="0 0 38.0e-3"/>
+        <geometry>
+          <cylinder radius="51.500e-3" length="76.0e-3" />
+        </geometry>
+      </collision>
+    </link>
+    <link name="${lidar_frame}"/>
+    <joint name="${prefix}hesai_base_to_${lidar_frame}" type="fixed">
+      <!-- See XT32 user manual -->
+      <origin xyz="0.0 0.0 46.4e-3" rpy="0.0 0.0 ${pi/2}"/>
+      <parent link="${prefix}hesai_base"/>
+      <child link="${lidar_frame}" />
+    </joint>
+    <xacro:if value="${simulation}">
+      <xacro:include filename="$(find hesai_description)/urdf/gazebo.urdf.xacro"/>
+      <xacro:hesai_gazebo prefix="${prefix}" lidar_frame="${lidar_frame}" topic_name="${topic_name}" min_range="0.4" max_range="80.0"
+        min_horizontal_angle="-180.0" max_horizontal_angle="180.0" min_vertical_angle="-16.0" max_vertical_angle="15.0"
+        hz="10" samples="2000" lasers="32" collision_range="0.3" noise="0.008" use_gpu="${use_gpu}"
+      />
+    </xacro:if>
+  </xacro:macro>
 </robot>

File: urdf/hesai_xt32_standalone.urdf.xacro (robot description, xacro)
@@ -1,24 +1,12 @@
 <?xml version="1.0"?>
-<!-- Copyright 2022 University of Oxford
-   Licensed under the Apache License, Version 2.0 (the "License");
-   you may not use this file except in compliance with the License.
-   You may obtain a copy of the License at
-       http://www.apache.org/licenses/LICENSE-2.0
-   Unless required by applicable law or agreed to in writing, software
-   distributed under the License is distributed on an "AS IS" BASIS,
-   WITHOUT WARRANTIES OR CONDITIONS OF ANY KIND, either express or implied.
-   See the License for the specific language governing permissions and
-   limitations under the License. -->
 <robot name="hesai" xmlns:xacro="http://www.ros.org/wiki/xacro">
-  <xacro:include filename="$(find hesai_description)/urdf/hesai_xt32.urdf.xacro" />
   <xacro:arg name="prefix" default="" />
   <xacro:arg name="simulation" default="false" />
   <xacro:arg name="use_gpu" default="true" />
-  <!-- Dummy link  -->
+  <xacro:include filename="$(find hesai_description)/urdf/hesai_xt32.urdf.xacro" />
   <link name="base"/>
-  <xacro:hesai_xt32_device parent="base" prefix="$(arg prefix)"
-    lidar_frame="$(arg prefix)pandar"
-    simulation="$(arg simulation)" use_gpu="$(arg use_gpu)" >
+  <xacro:hesai_xt32 parent="base" prefix="$(arg prefix)" lidar_frame="$(arg prefix)pandar"
+                    simulation="$(arg simulation)" use_gpu="$(arg use_gpu)" >
     <origin xyz="0 0 0" rpy="0 0 0" />
-  </xacro:hesai_xt32_device>
+  </xacro:hesai_xt32>
 </robot>
