Commit message: feat: Add Gazebo Classic simulation

File: urdf/gazebo.urdf.xacro (robot description, xacro)
@@ -4,18 +4,13 @@
                min_range:=0.4 max_range:=80.0 min_horizontal_angle:=-180.0 max_horizontal_angle:=180.0
                min_vertical_angle:=-16.0 max_vertical_angle:=15.0 hz:=10 samples:=2000 lasers:=32
-               collision_range:=0.3 noise:=0.008 visualize:=false use_gpu:=true">
+               collision_range:=0.3 noise:=0.008 visualize:=false">
     <gazebo reference="${lidar_frame}">
-      <xacro:if value="${use_gpu}">
-        <xacro:property name="ray_type" value="gpu_ray" />
-        <xacro:property name="laser_plugin" value="libgazebo_ros_velodyne_gpu_laser.so" />
-      </xacro:if>
-      <xacro:unless value="${use_gpu}">
-        <xacro:property name="ray_type" value="ray" />
-        <xacro:property name="laser_plugin" value="libgazebo_ros_velodyne_laser.so" />
-      </xacro:unless>
-      <sensor type="${ray_type}" name="${prefix}hesai_sensor">
-        <pose>0 0 0 0 0 0</pose>
+      <sensor name="${prefix}hesai_sensor" type="lidar">
+        <update_rate>${hz}</update_rate>
         <visualize>${visualize}</visualize>
-        <update_rate>${hz}</update_rate>
+        <always_on>true</always_on>
+        <ignition_frame_id>${lidar_frame}</ignition_frame_id>
+        <topic>${topic_name}</topic>
+        <!-- 'ray' for Gazebo Classic, 'lidar' for Ignition -->
         <ray>
           <scan>
@@ -36,13 +31,11 @@
             <min>${collision_range}</min>
             <max>${max_range+1}</max>
-            <resolution>0.001</resolution>
+            <resolution>0.01</resolution>
           </range>
-          <noise>
-            <type>gaussian</type>
-            <mean>0.0</mean>
-            <stddev>0.0</stddev>
-          </noise>
         </ray>
-        <plugin name="${prefix}gazebo_ros_laser_controller" filename="${laser_plugin}">
+        <plugin name="${prefix}gazebo_ros_laser_controller" filename="libgazebo_ros_velodyne_laser.so">
+          <ros>
+            <remapping>~/out:=${topic_name}</remapping>
+          </ros>
           <topicName>${topic_name}</topicName>
           <frameName>${lidar_frame}</frameName>

File: urdf/hesai_qt64.urdf.xacro (robot description, xacro)
@@ -3,5 +3,5 @@
   <xacro:macro name="hesai_qt64" params="parent *origin prefix:='' name:=pandar_qt64
                                          topic_name:=/hesai/pandar
-                                         simulation:=false lidar_frame:=pandar use_gpu:=true">
+                                         simulation:=false lidar_frame:=pandar">
     <joint name="${parent}_to_${prefix}hesai" type="fixed">
       <xacro:insert_block name="origin"/>
@@ -41,5 +41,5 @@
       <xacro:hesai_gazebo prefix="${prefix}" lidar_frame="${lidar_frame}" topic_name="${topic_name}" min_range="0.1" max_range="20.0"
         min_horizontal_angle="-180.0" max_horizontal_angle="180.0" min_vertical_angle="-52.1" max_vertical_angle="52.1"
-        hz="10" samples="600" lasers="64" collision_range="0.3" noise="0.008" use_gpu="${use_gpu}"
+        hz="10" samples="600" lasers="64" collision_range="0.3" noise="0.008"
       />
     </xacro:if>

File: urdf/hesai_qt64_standalone.urdf.xacro (robot description, xacro)
@@ -3,9 +3,8 @@
   <xacro:arg name="prefix" default="" />
   <xacro:arg name="simulation" default="false" />
-  <xacro:arg name="use_gpu" default="true" />
   <xacro:include filename="$(find hesai_description)/urdf/hesai_qt64.urdf.xacro" />
   <link name="base"/>
   <xacro:hesai_qt64 parent="base" prefix="$(arg prefix)" lidar_frame="$(arg prefix)pandar"
-                    simulation="$(arg simulation)" use_gpu="$(arg use_gpu)" >
+                    simulation="$(arg simulation)" >
     <origin xyz="0 0 0" rpy="0 0 0" />
   </xacro:hesai_qt64>

File: urdf/hesai_xt32.urdf.xacro (robot description, xacro)
@@ -3,5 +3,5 @@
   <xacro:macro name="hesai_xt32" params="parent *origin prefix:='' name:=hesai_xt32
                                         topic_name:=/hesai/pandar
-                                        simulation:=false lidar_frame:=pandar use_gpu:=true">
+                                        simulation:=false lidar_frame:=pandar">
     <joint name="${parent}_to_${prefix}hesai" type="fixed">
       <xacro:insert_block name="origin"/>
@@ -42,5 +42,5 @@
       <xacro:hesai_gazebo prefix="${prefix}" lidar_frame="${lidar_frame}" topic_name="${topic_name}" min_range="0.4" max_range="80.0"
         min_horizontal_angle="-180.0" max_horizontal_angle="180.0" min_vertical_angle="-16.0" max_vertical_angle="15.0"
-        hz="10" samples="2000" lasers="32" collision_range="0.3" noise="0.008" use_gpu="${use_gpu}"
+        hz="10" samples="2000" lasers="32" collision_range="0.3" noise="0.008"
       />
     </xacro:if>

File: urdf/hesai_xt32_standalone.urdf.xacro (robot description, xacro)
@@ -3,9 +3,8 @@
   <xacro:arg name="prefix" default="" />
   <xacro:arg name="simulation" default="false" />
-  <xacro:arg name="use_gpu" default="true" />
   <xacro:include filename="$(find hesai_description)/urdf/hesai_xt32.urdf.xacro" />
   <link name="base"/>
   <xacro:hesai_xt32 parent="base" prefix="$(arg prefix)" lidar_frame="$(arg prefix)pandar"
-                    simulation="$(arg simulation)" use_gpu="$(arg use_gpu)" >
+                    simulation="$(arg simulation)" >
     <origin xyz="0 0 0" rpy="0 0 0" />
   </xacro:hesai_xt32>

Commit message: Revert "Add support for Gazebo Classic simulation"

File: urdf/gazebo.urdf.xacro (robot description, xacro)
@@ -4,13 +4,18 @@
                min_range:=0.4 max_range:=80.0 min_horizontal_angle:=-180.0 max_horizontal_angle:=180.0
                min_vertical_angle:=-16.0 max_vertical_angle:=15.0 hz:=10 samples:=2000 lasers:=32
-               collision_range:=0.3 noise:=0.008 visualize:=false">
+               collision_range:=0.3 noise:=0.008 visualize:=false use_gpu:=true">
     <gazebo reference="${lidar_frame}">
-      <sensor name="${prefix}hesai_sensor" type="lidar">
+      <xacro:if value="${use_gpu}">
+        <xacro:property name="ray_type" value="gpu_ray" />
+        <xacro:property name="laser_plugin" value="libgazebo_ros_velodyne_gpu_laser.so" />
+      </xacro:if>
+      <xacro:unless value="${use_gpu}">
+        <xacro:property name="ray_type" value="ray" />
+        <xacro:property name="laser_plugin" value="libgazebo_ros_velodyne_laser.so" />
+      </xacro:unless>
+      <sensor type="${ray_type}" name="${prefix}hesai_sensor">
+        <pose>0 0 0 0 0 0</pose>
+        <visualize>${visualize}</visualize>
         <update_rate>${hz}</update_rate>
-        <visualize>${visualize}</visualize>
-        <always_on>true</always_on>
-        <ignition_frame_id>${lidar_frame}</ignition_frame_id>
-        <topic>${topic_name}</topic>
-        <!-- 'ray' for Gazebo Classic, 'lidar' for Ignition -->
         <ray>
           <scan>
@@ -31,11 +36,13 @@
             <min>${collision_range}</min>
             <max>${max_range+1}</max>
-            <resolution>0.01</resolution>
+            <resolution>0.001</resolution>
           </range>
+          <noise>
+            <type>gaussian</type>
+            <mean>0.0</mean>
+            <stddev>0.0</stddev>
+          </noise>
         </ray>
-        <plugin name="${prefix}gazebo_ros_laser_controller" filename="libgazebo_ros_velodyne_laser.so">
-          <ros>
-            <remapping>~/out:=${topic_name}</remapping>
-          </ros>
+        <plugin name="${prefix}gazebo_ros_laser_controller" filename="${laser_plugin}">
           <topicName>${topic_name}</topicName>
           <frameName>${lidar_frame}</frameName>

File: urdf/hesai_qt64.urdf.xacro (robot description, xacro)
@@ -3,5 +3,5 @@
   <xacro:macro name="hesai_qt64" params="parent *origin prefix:='' name:=pandar_qt64
                                          topic_name:=/hesai/pandar
-                                         simulation:=false lidar_frame:=pandar">
+                                         simulation:=false lidar_frame:=pandar use_gpu:=true">
     <joint name="${parent}_to_${prefix}hesai" type="fixed">
       <xacro:insert_block name="origin"/>
@@ -41,5 +41,5 @@
       <xacro:hesai_gazebo prefix="${prefix}" lidar_frame="${lidar_frame}" topic_name="${topic_name}" min_range="0.1" max_range="20.0"
         min_horizontal_angle="-180.0" max_horizontal_angle="180.0" min_vertical_angle="-52.1" max_vertical_angle="52.1"
-        hz="10" samples="600" lasers="64" collision_range="0.3" noise="0.008"
+        hz="10" samples="600" lasers="64" collision_range="0.3" noise="0.008" use_gpu="${use_gpu}"
       />
     </xacro:if>

File: urdf/hesai_qt64_standalone.urdf.xacro (robot description, xacro)
@@ -3,8 +3,9 @@
   <xacro:arg name="prefix" default="" />
   <xacro:arg name="simulation" default="false" />
+  <xacro:arg name="use_gpu" default="true" />
   <xacro:include filename="$(find hesai_description)/urdf/hesai_qt64.urdf.xacro" />
   <link name="base"/>
   <xacro:hesai_qt64 parent="base" prefix="$(arg prefix)" lidar_frame="$(arg prefix)pandar"
-                    simulation="$(arg simulation)" >
+                    simulation="$(arg simulation)" use_gpu="$(arg use_gpu)" >
     <origin xyz="0 0 0" rpy="0 0 0" />
   </xacro:hesai_qt64>

File: urdf/hesai_xt32.urdf.xacro (robot description, xacro)
@@ -3,5 +3,5 @@
   <xacro:macro name="hesai_xt32" params="parent *origin prefix:='' name:=hesai_xt32
                                         topic_name:=/hesai/pandar
-                                        simulation:=false lidar_frame:=pandar">
+                                        simulation:=false lidar_frame:=pandar use_gpu:=true">
     <joint name="${parent}_to_${prefix}hesai" type="fixed">
       <xacro:insert_block name="origin"/>
@@ -42,5 +42,5 @@
       <xacro:hesai_gazebo prefix="${prefix}" lidar_frame="${lidar_frame}" topic_name="${topic_name}" min_range="0.4" max_range="80.0"
         min_horizontal_angle="-180.0" max_horizontal_angle="180.0" min_vertical_angle="-16.0" max_vertical_angle="15.0"
-        hz="10" samples="2000" lasers="32" collision_range="0.3" noise="0.008"
+        hz="10" samples="2000" lasers="32" collision_range="0.3" noise="0.008" use_gpu="${use_gpu}"
       />
     </xacro:if>

File: urdf/hesai_xt32_standalone.urdf.xacro (robot description, xacro)
@@ -3,8 +3,9 @@
   <xacro:arg name="prefix" default="" />
   <xacro:arg name="simulation" default="false" />
+  <xacro:arg name="use_gpu" default="true" />
   <xacro:include filename="$(find hesai_description)/urdf/hesai_xt32.urdf.xacro" />
   <link name="base"/>
   <xacro:hesai_xt32 parent="base" prefix="$(arg prefix)" lidar_frame="$(arg prefix)pandar"
-                    simulation="$(arg simulation)" >
+                    simulation="$(arg simulation)" use_gpu="$(arg use_gpu)" >
     <origin xyz="0 0 0" rpy="0 0 0" />
   </xacro:hesai_xt32>

Commit message: Change pandar frame to hesai_lidar to match ros2 driver

File: urdf/gazebo.urdf.xacro (robot description, xacro)
@@ -1,5 +1,5 @@
 <?xml version="1.0"?>
 <robot xmlns:xacro="http://www.ros.org/wiki/xacro">
-  <xacro:macro name="hesai_gazebo" params="prefix lidar_frame:=pandar topic_name=/hesai/pandar
+  <xacro:macro name="hesai_gazebo" params="prefix lidar_frame:=hesai_lidar topic_name=/hesai/pandar
                min_range:=0.4 max_range:=80.0 min_horizontal_angle:=-180.0 max_horizontal_angle:=180.0
                min_vertical_angle:=-16.0 max_vertical_angle:=15.0 hz:=10 samples:=2000 lasers:=32

File: urdf/hesai_qt64.urdf.xacro (robot description, xacro)
@@ -1,7 +1,7 @@
 <?xml version="1.0"?>
 <robot name="hesai_qt64" xmlns:xacro="http://www.ros.org/wiki/xacro">
-  <xacro:macro name="hesai_qt64" params="parent *origin prefix:='' name:=pandar_qt64
+  <xacro:macro name="hesai_qt64" params="parent *origin prefix:='' name:=hesai_lidar_qt64
                                          topic_name:=/hesai/pandar
-                                         simulation:=false lidar_frame:=pandar use_gpu:=true">
+                                         simulation:=false lidar_frame:=hesai_lidar use_gpu:=true">
     <joint name="${parent}_to_${prefix}hesai" type="fixed">
       <xacro:insert_block name="origin"/>

File: urdf/hesai_qt64_standalone.urdf.xacro (robot description, xacro)
@@ -6,5 +6,5 @@
   <xacro:include filename="$(find hesai_description)/urdf/hesai_qt64.urdf.xacro" />
   <link name="base"/>
-  <xacro:hesai_qt64 parent="base" prefix="$(arg prefix)" lidar_frame="$(arg prefix)pandar"
+  <xacro:hesai_qt64 parent="base" prefix="$(arg prefix)" lidar_frame="$(arg prefix)hesai_lidar"
                     simulation="$(arg simulation)" use_gpu="$(arg use_gpu)" >
     <origin xyz="0 0 0" rpy="0 0 0" />

File: urdf/hesai_xt32.urdf.xacro (robot description, xacro)
@@ -3,5 +3,5 @@
   <xacro:macro name="hesai_xt32" params="parent *origin prefix:='' name:=hesai_xt32
                                         topic_name:=/hesai/pandar
-                                        simulation:=false lidar_frame:=pandar use_gpu:=true">
+                                        simulation:=false lidar_frame:=hesai_lidar use_gpu:=true">
     <joint name="${parent}_to_${prefix}hesai" type="fixed">
       <xacro:insert_block name="origin"/>

File: urdf/hesai_xt32_standalone.urdf.xacro (robot description, xacro)
@@ -6,5 +6,5 @@
   <xacro:include filename="$(find hesai_description)/urdf/hesai_xt32.urdf.xacro" />
   <link name="base"/>
-  <xacro:hesai_xt32 parent="base" prefix="$(arg prefix)" lidar_frame="$(arg prefix)pandar"
+  <xacro:hesai_xt32 parent="base" prefix="$(arg prefix)" lidar_frame="$(arg prefix)hesai_lidar"
                     simulation="$(arg simulation)" use_gpu="$(arg use_gpu)" >
     <origin xyz="0 0 0" rpy="0 0 0" />
