Commit message: use package:// rather than file:// so models load over network

File: urdf/hesai_qt64.urdf.xacro (robot description, xacro)
@@ -13,5 +13,5 @@
         <origin xyz="0 0 0" rpy="0 0 0" />
         <geometry>
-          <mesh filename="file://$(find hesai_description)/meshes/visual/qt64.dae" />
+          <mesh filename="package://hesai_description/meshes/visual/qt64.dae" />
         </geometry>
       </visual>

File: urdf/hesai_xt32.urdf.xacro (robot description, xacro)
@@ -13,5 +13,5 @@
         <origin xyz="0 0 0" rpy="0 0 0" />
         <geometry>
-          <mesh filename="file://$(find hesai_description)/meshes/visual/xt32.dae" />
+          <mesh filename="package://hesai_description/meshes/visual/xt32.dae" />
         </geometry>
       </visual>

Commit message: Reverse unnecessarry search & replace change

File: urdf/hesai_qt64.urdf.xacro (robot description, xacro)
@@ -1,5 +1,5 @@
 <?xml version="1.0"?>
 <robot name="hesai_qt64" xmlns:xacro="http://www.ros.org/wiki/xacro">
-  <xacro:macro name="hesai_qt64" params="parent *origin prefix:='' name:=hesai_lidar_qt64
+  <xacro:macro name="hesai_qt64" params="parent *origin prefix:='' name:=pandar_qt64
                                          topic_name:=/hesai/pandar
                                          simulation:=false lidar_frame:=hesai_lidar use_gpu:=true">
